Commit message: ewew

File: src/el5206_description/urdf/common_properties.xacro (robot description, xacro)
@@ -15,5 +15,5 @@
   </material>
   <material name="green">
-    <color rgba="0.0 0.8 0.0 1.0"/>
+    <color rgba="0.0 0.4 0.0 1.0"/>
   </material>
   <material name="grey">
@@ -27,5 +27,5 @@
   </material>
   <material name="red">
-    <color rgba="0.8 0.0 0.0 1.0"/>
+    <color rgba="1.0 0.0 0.0 1.0"/>
   </material>
   <material name="white">

File: src/el5206_description/urdf/turtlebot3_burger.gazebo.xacro (robot description, xacro)
@@ -3,6 +3,7 @@
   <xacro:arg name="laser_visual" default="false"/>
   <xacro:arg name="imu_visual"   default="false"/>
+<!-- uwu -->
   <gazebo reference="base_link">
-    <material>Gazebo/DarkGrey</material>
+    <material>Gazebo/Green</material>
   </gazebo>
   <gazebo reference="wheel_left_link">
@@ -136,3 +137,33 @@
     </sensor>
   </gazebo>
+  <!-- uwu -->
+  <gazebo reference="camera_link">
+    <material>Gazebo/Red</material>
+    <sensor name="camera_link_camera" type="depth">
+    <pose> 0 0 0 0 0 0 </pose>
+    <visualize>true</visualize>
+    <update_rate>20</update_rate>
+    <camera>
+      <horizontal_fov>1.089</horizontal_fov>
+      <image>
+        <format>R8G8B8</format>
+        <width>640</width>
+        <height>480</height>
+      </image>
+      <clip>
+        <near>0.05</near>
+        <far>8.0</far>
+      </clip>
+    </camera>
+    <plugin name="camera_controller" filename="libgazebo_ros_camera.so">
+        <baseline>0.2</baseline>
+        <alwaysOn>true</alwaysOn>
+        <updateRate>1.0</updateRate>
+        <cameraName>camera_link_camera</cameraName>
+        <imageTopicName>camera_link_camera/color/image_raw</imageTopicName>
+        <cameraInfoTopicName>camera_link_camera/color/camera_info</cameraInfoTopicName>
+        <frame_name>camera_link_optical</frame_name>
+    </plugin> -->
+</sensor>
+</gazebo>
 </robot>
